File: kicad/rev1.1b/megaflash.kicad_pcb (KiCad board)
At the start: 2 copper layers, 102 x 52 mm, 22 parts, among them J1 EXPSLOT, U1 74LVC8T245, U2 74LVC8T245, U3 GAL16V8, U4 Pico, U5 W25Q01JVSF, U6 W25Q01JVSF

Commit message: Revised Rev1.1b PCB
Parts:
- renumbered C5 to C4, C6 to C5, C7 to C6, C8 to C7
Changed lines of the file:
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@@
 		(descr "C, Disc series, Radial, pin pitch=5.00mm, diameter*width=5.1*3.2mm^2, Capacitor, http://www.vishay.com/docs/45233/krseries.pdf")
 		(tags "C Disc series Radial pin pitch 5.00mm diameter 5.1mm width 3.2mm Capacitor")
-		(property "Reference" "C7"
+		(property "Reference" "C6"
 			(at 7.535 0 0)
 			(layer "F.SilkS")
@@
 		(descr "C, Disc series, Radial, pin pitch=5.00mm, diameter*width=5.1*3.2mm^2, Capacitor, http://www.vishay.com/docs/45233/krseries.pdf")
 		(tags "C Disc series Radial pin pitch 5.00mm diameter 5.1mm width 3.2mm Capacitor")
-		(property "Reference" "C8"
+		(property "Reference" "C7"
 			(at -2.58 0 0)
 			(layer "F.SilkS")
@@
 		(descr "C, Disc series, Radial, pin pitch=5.00mm, diameter*width=5.1*3.2mm^2, Capacitor, http://www.vishay.com/docs/45233/krseries.pdf")
 		(tags "C Disc series Radial pin pitch 5.00mm diameter 5.1mm width 3.2mm Capacitor")
-		(property "Reference" "C6"
+		(property "Reference" "C5"
 			(at 2.5 3.175 0)
 			(layer "F.SilkS")
@@
 		(descr "C, Disc series, Radial, pin pitch=5.00mm, diameter*width=5.1*3.2mm^2, Capacitor, http://www.vishay.com/docs/45233/krseries.pdf")
 		(tags "C Disc series Radial pin pitch 5.00mm diameter 5.1mm width 3.2mm Capacitor")
-		(property "Reference" "C5"
+		(property "Reference" "C4"
 			(at 7.58 0 0)
 			(layer "F.SilkS")

Commit message: Revised PCB Rev 1.1B
Parts:
- moved R2 23.1 mm to (166.8, 88.9)
- moved R1 23.1 mm to (166.8, 92.3)
- moved U5 17.0 mm to (161.7, 72.5)
- moved C6 17.0 mm to (159.4, 64.6)
- moved D2 6.67 mm to (72.4, 47.0), turned to 180 degrees
- moved J1 6.06 mm to (71.6, 93.7)
- moved H1 6.00 mm to (162.4, 82.2)
- moved D1 5.09 mm to (78.7, 47.3)
- moved U6 0.50 mm to (161.7, 55.6)
Routing:
- net +3.3V: track 166.4 -> 188.9 mm, vias 3 -> 4
- net /SPI0_RX: track 43.5 -> 29.7 mm, vias 3 -> 0
- net /R/~{W}#: track 59.1 -> 46.1 mm, vias 4 -> 1
- net /~{SPI0_CS1}: track 43.7 -> 55.6 mm, vias 2 -> 1
- net /BUF_DIR#: track 52.6 -> 42.7 mm, vias 4 -> 1
- net /A12#: track 32.5 -> 23.0 mm, vias 2 -> 1
- net /A10#: track 24.9 -> 16.2 mm
- net /~{SPI0_CS0}: track 32.7 -> 24.3 mm, vias 2 -> 1
- net /SPI0_TX: track 53.6 -> 45.4 mm, vias 2 -> 0
- net /A14#: track 36.7 -> 28.5 mm
- net /A9#: track 16.4 -> 9.18 mm, vias 2 -> 0
- net /A13#: track 36.9 -> 30.1 mm
- net /A7#: track 9.56 -> 16.0 mm, vias 0 -> 1
- net /A15#: track 30.2 -> 24.5 mm, vias 2 -> 1
- net /A4#: track 24.3 -> 30.0 mm
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