File: kicad/rev1.1b/megaflash.kicad_sch (KiCad schematic)
At the start: 22 parts, among them J1 EXPSLOT, U1 74LVC8T245, U2 74LVC8T245, U3 GAL16V8, U4 Pico, U5 W25Q01JVSF, U6 W25Q01JVSF

Commit message: Revised Rev1.1b PCB
Parts:
- renumbered C5 to C4, C6 to C5, C7 to C6, C8 to C7
